Commit message: added collision tags to gelslims and additional method for adding objects to the world via yumi

File: src/airobot/urdfs/yumi_gelsight.urdf (robot description, URDF)
Before this commit: robot yumi, 29 links, 28 joints
Links:
- link table_top: geometry collision mesh filename=meshes/table/table_top.stl; visual mesh filename=meshes/table/table_top.stl
- link yumi_gel_l: geometry collision mesh filename=meshes/mpalm/mpalms_gel.stl; visual mesh filename=meshes/mpalm/mpalms_gel.stl
- link yumi_gel_r: geometry collision mesh filename=meshes/mpalm/mpalms_gel.stl; visual mesh filename=meshes/mpalm/mpalms_gel.stl
- link yumi_metal_bottom_l: geometry collision mesh filename=meshes/mpalm/mpalms_shield.stl; visual mesh filename=meshes/mpalm/mpalms_shield.stl
- link yumi_metal_bottom_r: geometry collision mesh filename=meshes/mpalm/mpalms_shield.stl; visual mesh filename=meshes/mpalm/mpalms_shield.stl
- link yumi_palm_body_l: geometry collision mesh filename=meshes/mpalm/mpalms_body.stl; visual mesh filename=meshes/mpalm/mpalms_body.stl
- link yumi_palm_body_r: geometry collision mesh filename=meshes/mpalm/mpalms_body.stl; visual mesh filename=meshes/mpalm/mpalms_body.stl
- link yumi_palm_l: geometry collision mesh filename=meshes/mpalm/mpalms_top.stl; visual mesh filename=meshes/mpalm/mpalms_top.stl
- link yumi_palm_r: geometry collision mesh filename=meshes/mpalm/mpalms_top.stl; visual mesh filename=meshes/mpalm/mpalms_top.stl
- link yumi_rail_l: geometry collision mesh filename=meshes/mpalm/mpalms_rail.stl; visual mesh filename=meshes/mpalm/mpalms_rail.stl
- link yumi_rail_r: geometry collision mesh filename=meshes/mpalm/mpalms_rail.stl; visual mesh filename=meshes/mpalm/mpalms_rail.stl

Commit message: refactored for single arm and double arm base classes, and added nullspace option to single arm compute_ik. needs debugging

File: src/airobot/urdfs/yumi_gelsight.urdf (robot description, URDF)
Before this commit: robot yumi, 29 links, 28 joints
Joints:
- joint yumi_gel_l: limit lower=-0.0025 upper=0.0025 -> lower=0 upper=0.0025
- joint yumi_gel_r: limit lower=-0.0025 upper=0.0025 -> lower=0 upper=0.00025
- joint yumi_palm_l: limit lower=0.0 upper=0.05 -> lower=0.0 upper=0.0075
- joint yumi_palm_r: limit lower=0.0 upper=0.05 -> lower=0.0 upper=0.0075
