Commit message: yumi palm and gripper classes working with some examples, palm urdf updated with prismatic joints at palm wrists

File: src/airobot/urdfs/yumi_gelslim_palm.urdf (robot description, URDF)
Before this commit: robot yumi, 29 links, 28 joints
Links:
- link table_top: geometry collision mesh filename=meshes/table/table_top.stl; visual mesh filename=meshes/table/table_top.stl
- link yumi_gel_l: geometry collision mesh filename=meshes/mpalm/mpalms_gel.stl; visual mesh filename=meshes/mpalm/mpalms_gel.stl
- link yumi_gel_r: geometry collision mesh filename=meshes/mpalm/mpalms_gel.stl; visual mesh filename=meshes/mpalm/mpalms_gel.stl
Joints:
- joint yumi_gel_l: axis (none) -> 0 1 0 ; limit (none) -> lower=0 upper=0.0025; type fixed -> prismatic
- joint yumi_gel_r: axis (none) -> 0 1 0 ; limit (none) -> lower=0 upper=0.00025; type fixed -> prismatic
- joint yumi_palm_l: axis (none) -> 0 1 0 ; limit (none) -> lower=0.0 upper=0.0075; type fixed -> prismatic
- joint yumi_palm_r: axis (none) -> 0 1 0 ; limit (none) -> lower=0.0 upper=0.0075; type fixed -> prismatic

Commit message: added ur5e with stick ee to cfgs and urdfs, and updated yumi palm urdf with smaller link masses and new joint torques

File: src/airobot/urdfs/yumi_gelslim_palm.urdf (robot description, URDF)
Before this commit: robot yumi, 29 links, 28 joints
Links:
- link yumi_gel_l: mass 2 -> 0.01
- link yumi_gel_r: mass 2 -> 0.01
- link yumi_metal_bottom_l: mass 2 -> 0.3
- link yumi_metal_bottom_r: mass 2 -> 0.3
- link yumi_palm_body_l: mass None -> 0.02
- link yumi_palm_body_r: mass None -> 0.02
- link yumi_palm_l: mass 2 -> 0.3
- link yumi_palm_r: mass 2 -> 0.1
- link yumi_rail_l: mass None -> 0.02
- link yumi_rail_r: mass None -> 0.02
- link yumi_tip_l: mass None -> 0.001
- link yumi_tip_r: mass None -> 0.001
