Commit message: updated ur5e_stick with offset end effector and ee_link_name in cfg file

File: src/airobot/urdfs/ur5e_stick_pybullet.urdf (robot description, URDF)
Before this commit: robot ur5e, 13 links, 12 joints
Links:
- removed link gripper_tip
- added link stick_tip
- link ee_stick: geometry collision mesh filename=meshes/custom_ee_tools/stick/visual/ur5e_ee_stick.stl scale=0.001 0.001 0.001; visual mesh filename=meshes/custom_ee_tools/stick/visual/ur5e_ee_stick.stl scale=0.001 0.001 0.001
Joints:
- removed joint gripper_tip_joint
- added joint stick_tip_joint: type fixed, parent ee_stick, child stick_tip, origin xyz= 0.00 0.0 0.1524 rpy=0.0 0.0 0.0
- joint stick_joint: parent gripper_tip -> tool0

Commit message: Update ur5e_stick_pybullet.urdf

File: src/airobot/urdfs/ur5e_stick_pybullet.urdf (robot description, URDF)
Before this commit: robot ur5e, 13 links, 12 joints
Links:
- removed link stick_tip
- added link ee_tip
Joints:
- removed joint stick_tip_joint
- added joint ee_tip_joint: type fixed, parent ee_stick, child ee_tip, origin xyz= 0.00 0.0 0.1524 rpy=0.0 0.0 0.0
