Commit message: Update ur5e_pybullet.urdf

File: src/airobot/urdfs/ur5e_pybullet.urdf (robot description, URDF)
Before this commit: robot ur5e, 12 links, 11 joints
Links:
- removed link gripper_tip
- added link ee_tip
Joints:
- removed joint gripper_tip_joint
- added joint ee_tip_joint: type fixed, parent tool0, child ee_tip, origin xyz= 0.00 0.0 0.0 rpy=0.0 0.0 0.0
